File: pcb.kicad_pcb (KiCad board)
At the start: 2 copper layers, 247.7 x 95.2 mm, 86 parts, among them SW1 SW_PUSH, SW10 SW_PUSH, SW11 SW_PUSH, SW12 SW_PUSH, SW13 SW_PUSH, SW14 SW_PUSH, SW15 SW_PUSH, SW16 SW_PUSH, SW17 SW_PUSH, SW18 SW_PUSH, SW19 SW_PUSH, SW2 SW_PUSH, SW20 SW_PUSH, SW21 SW_PUSH, SW22 SW_PUSH, SW23 SW_PUSH, SW24 SW_PUSH, SW25 SW_PUSH, SW26 SW_PUSH, SW27 SW_PUSH, SW28 SW_PUSH, SW29 SW_PUSH, SW3 SW_PUSH, SW30 SW_PUSH, SW31 SW_PUSH, SW32 SW_PUSH, SW33 SW_PUSH, SW34 SW_PUSH, SW35 SW_PUSH, SW36 SW_PUSH, SW37 SW_PUSH, SW38 SW_PUSH, SW39 SW_PUSH, SW4 SW_PUSH, SW40 SW_PUSH, SW41 SW_PUSH, SW42 SW_PUSH, SW5 SW_PUSH, SW6 SW_PUSH, SW7 SW_PUSH, SW8 SW_PUSH, SW9 SW_PUSH, U1 ProMicro

Commit message: refactored wiring
Parts:
- moved RSSW0 3.57 mm to (152.4, 80.5)
Routing:
- net ROW6: track 129.2 -> 144.4 mm
- net ROW5: track 113.0 -> 124.4 mm
- net ROW7: track 88.7 -> 100.1 mm
- net ROW1: track 145.2 -> 156.0 mm, vias 1 -> 0
- net GND: track 55.4 -> 44.9 mm, vias 1 -> 0
- net Net-(U1-RST): track 38.2 -> 31.0 mm
- net ROW4: track 116.8 -> 120.9 mm
- net COL0: track 245.7 -> 249.5 mm
- net ROW2: track 162.3 -> 165.9 mm, vias 1 -> 0
- net COL2: track 248.5 -> 244.9 mm
- net ROW3: track 121.6 -> 125.0 mm, vias 1 -> 0
- net COL1: track 249.4 -> 246.3 mm
- net COL3: track 250.1 -> 247.7 mm
- net ROW0: track 130.5 -> 132.3 mm
- net COL4: track 248.0 -> 246.6 mm
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
Commit message: set hole
Parts:
- added Ref**: Val**, kbd:spacer_m2, F.Cu at (47.6, 44.8)
- added Ref**: Val**, kbd:spacer_m2, F.Cu at (257.2, 63.8)
- added Ref**: Val**, kbd:spacer_m2, F.Cu at (123.8, 47.1)
- added Ref**: Val**, kbd:spacer_m2, F.Cu at (181.0, 103.1)
- added Ref**: Val**, kbd:spacer_m2, F.Cu at (47.6, 63.8)
- added Ref**: Val**, kbd:spacer_m2, F.Cu at (85.7, 68.6)
- added Ref**: Val**, kbd:spacer_m2, F.Cu at (123.8, 103.1)
- added Ref**: Val**, kbd:spacer_m2, F.Cu at (219.1, 68.6)
- added Ref**: Val**, kbd:spacer_m2, F.Cu at (257.2, 44.8)
- added Ref**: Val**, kbd:spacer_m2, F.Cu at (181.0, 47.1)
Routing:
- net COL1: track 246.3 -> 246.9 mm
- net COL5: track 246.9 -> 247.5 mm
- net COL0: track 249.5 -> 250.0 mm

Commit message: create garbar file
Routing:
- net GND: track 44.9 -> 0.00 mm
- net ROW0: track 132.7 -> 175.2 mm, vias 1 -> 0
- net ROW4: track 120.9 -> 118.2 mm
- net Net-(U1-RST): track 31.0 -> 28.7 mm
- net COL1: track 246.9 -> 244.9 mm
- net COL3: track 248.2 -> 249.9 mm
- net COL4: track 246.6 -> 248.2 mm
- net ROW1: track 156.1 -> 157.5 mm
- net ROW5: track 124.3 -> 125.6 mm
- net ROW6: track 144.4 -> 143.2 mm
- net COL0: track 250.0 -> 251.0 mm
- net ROW7: track 100.1 -> 99.2 mm
- added copper zone on B.Cu, net GND
- added copper zone on F.Cu, net GND
Other:
- board text added: "Maggie42 ver.1.0 Tamaroh"
